File: .history/mezclador doble canal.kicad_pcb (KiCad board)
At the start: 2 copper layers, 55 x 50.1 mm, 40 parts, among them J1 Conn_Coaxial, J3 Conn_Coaxial, J4 Conn_Coaxial, J5 Conn_Coaxial, J7 Screw_Terminal_01x02, J8 Conn_Coaxial, SW1 SW_SPST, U1 NE5532, U2 TL071

Commit message: eliminando RV1 no necesario
Parts:
- removed RV1: R_Potentiometer, personal:potentiometer pads
Connections:
- C6 pad 2: Net-(C6-Pad2) -> Net-(C3-Pad2)
- RV4 pad 2: Net-(C6-Pad2) -> Net-(C3-Pad2)
Routing:
- net Net-(C3-Pad2): track 8.78 -> 43.3 mm
- net Net-(C2-Pad2): track 116.5 -> 82.3 mm
- net GND: track 334.8 -> 325.8 mm
- net Net-(C6-Pad2): track 7.62 -> 0.00 mm
